File: SabidosReceiver.kicad_sch (KiCad schematic)
At the start: 79 parts, among them Q1 2N7002, Q2 2N7002, U2 PT2322-S, U3 PT2323-S

Commit message: Complete PT2323 stereo inputs and correct center audio path
Connections:
- net SELECTOR-CTO is gone; now on net SELECTOR-CT: R35.1
- net PT1L: now reaches U3.1 (L1)
- net PT2L: now reaches U3.2 (L2)
- net PT4R: now reaches U3.25 (R4)
- net PT3R: now reaches U3.26 (R3)
- net PT2R: now reaches U3.27 (R2)
- net PT1R: now reaches U3.28 (R1)
- net PT3L: now reaches U3.3 (L3)
- net PT4L: now reaches U3.4 (L4)
Other:
- added sheet Entradas Stereo (entradas_estereo.kicad_sch)
Changed lines of the file:
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@@
 		)
 	)
-	(label "SELECTOR-CTO"
+	(label "SELECTOR-CT"
 		(at 138.43 201.93 0)
 		(effects
@@
 	)
 	(embedded_fonts no)
+(global_label "PT1L" (shape input) (at 49.53 195.58 0) (effects (font (size 0.85 0.85)) (justify right)))
+(global_label "PT1R" (shape input) (at 90.17 195.58 180) (effects (font (size 0.85 0.85)) (justify left)))
+(global_label "PT2L" (shape input) (at 49.53 198.12 0) (effects (font (size 0.85 0.85)) (justify right)))
+(global_label "PT2R" (shape input) (at 90.17 198.12 180) (effects (font (size 0.85 0.85)) (justify left)))
+(global_label "PT3L" (shape input) (at 49.53 200.66 0) (effects (font (size 0.85 0.85)) (justify right)))
+(global_label "PT3R" (shape input) (at 90.17 200.66 180) (effects (font (size 0.85 0.85)) (justify left)))
+(global_label "PT4L" (shape input) (at 49.53 203.20 0) (effects (font (size 0.85 0.85)) (justify right)))
+(global_label "PT4R" (shape input) (at 90.17 203.20 180) (effects (font (size 0.85 0.85)) (justify left)))
+(sheet (at 175.26 250.19) (size 40.64 15.24) (stroke (width 0.1524) (type solid)) (fill (color 0 0 0 0))
+(property "Sheetname" "Entradas Stereo" (at 175.26 249 0) (effects (font (size 1.0 1.0))))
+(property "Sheetfile" "entradas_estereo.kicad_sch" (at 175.26 266.5 0) (effects (font (size 1.0 1.0))))
+(instances (project "SabidosReceiver" (path "/ac327e59-bfb2-4343-b248-420c1a5897eb" (page "6")))))
 )
